Commit message: last_updates

File: itu_agv_description/models/urdf/itu_agv_copy.xacro (robot description, xacro)
@@ -2,230 +2,100 @@
 <robot xmlns:xacro="http://wiki.ros.org/xacro"
   name="ITU_AGV">
-  <material name="blue">
-    <color rgba="0 0 0.8 1"/>
-  </material>
-  <link name="base_link">
-    <visual>
-       <origin xyz="0 0 0" rpy="0 0 0" />
+<joint name="AGV_1/base_joint" type="fixed">
+    <parent link="AGV_1/base_footprint"/>
+    <child link="AGV_1/base_link"/>
+    <origin xyz="0   0   0.12" rpy="0 0 0"/>
+    <axis xyz="0 0 0"/>
+    <limit lower="0" upper="0" effort="0" velocity="0"/>
+  </joint>
+  <joint name="AGV_1/base_to_wheel_left" type="fixed">
+    <parent link="AGV_1/base_link"/>
+    <child link="AGV_1/wheel_left"/>
+    <origin xyz="0    0.22 -0.02" rpy="1.571 0    0"/>
+    <axis xyz="0.e+00 -2.e-04 -1.e+00"/>
+    <limit lower="0" upper="0" effort="0" velocity="0"/>
+  </joint>
+  <joint name="AGV_1/base_to_wheel_right" type="fixed">
+    <parent link="AGV_1/base_link"/>
+    <child link="AGV_1/wheel_right"/>
+    <origin xyz="0   -0.22 -0.02" rpy="1.571 0    0"/>
+    <axis xyz="0.e+00 -2.e-04 -1.e+00"/>
+    <limit lower="0" upper="0" effort="0" velocity="0"/>
+  </joint>
+  <link name="AGV_1/base_link">
+    <inertial>
+      <mass value="5.67"/>
+      <origin xyz="0 0 0" rpy="0 0 0"/>
+      <inertia ixx="0.07" ixy="0" ixz="0" iyy="0.08" iyz="0" izz="0.10"/>
+    </inertial>
+    <collision name="AGV_1/collision">
+      <origin xyz="0    0   -0.11" rpy="0     0    -1.571"/>
       <geometry>
-        <mesh
-          filename="package://itu_agv_description/meshes/agv.dae"/>
+        <mesh filename="package://itu_agv_description/meshes/agv.stl" scale="1.0 1.0 1.0"/>
+      </geometry>
+    </collision>
+    <collision name="AGV_1/front_caster_collision">
+      <origin xyz="0.25  0   -0.07" rpy="0 0 0"/>
+      <geometry>
+        <sphere radius=".05"/>
+      </geometry>
+    </collision>
+    <collision name="AGV_1/back_caster_collision">
+      <origin xyz="-0.25  0   -0.07" rpy="0 0 0"/>
+      <geometry>
+        <sphere radius=".05"/>
+      </geometry>
+    </collision>
+    <visual name="AGV_1/visual">
+      <origin xyz="0    0   -0.11" rpy="0     0    -1.571"/>
+      <geometry>
+        <mesh filename="package://itu_agv_description/meshes/agv.stl" scale="1.0 1.0 1.0"/>
       </geometry>
     </visual>
-    <collision>
-    	<geometry>
-    	  <mesh
-          filename="package://itu_agv_description/meshes/agv.dae"/>
-    	</geometry>
-    </collision>
+    <visual name="AGV_1/front_caster_visual">
+      <origin xyz="0.25  0   -0.07" rpy="0 0 0"/>
+      <geometry>
+        <sphere radius=".05"/>
+      </geometry>
+    </visual>
+    <visual name="AGV_1/back_caster_visual">
+      <origin xyz="-0.25  0   -0.07" rpy="0 0 0"/>
+      <geometry>
+        <sphere radius=".05"/>
+      </geometry>
+    </visual>
+  </link>
+  <link name="AGV_1/base_footprint">
     <inertial>
-      <mass value="5"/>
-      <inertia ixx="0.07" ixy="0.0" ixz="0.0" iyy="0.08" iyz="0.0" izz="0.1"/>
+      <mass value="0"/>
+      <origin xyz="0 0 0" rpy="0 0 0"/>
+      <inertia ixx="0" ixy="0" ixz="0" iyy="0" iyz="0" izz="0"/>
     </inertial>
   </link>
-    <link name="front_caster">
-  	<visual>
-  		<pose xyz="0 0.25 0.05" rpy="0 0 0"/>
-  		<geometry>
-        	   <sphere radius="0.05"/>
-        	</geometry>
-        </visual>
-        <collision>
-        	<pose xyz="0 0.25 0.05" rpy="0 0 0"/>
-  		<geometry>
-        	   <sphere radius="0.05"/>
-        	</geometry>
-        </collision>
-   </link>
-   <joint name="base_link_to_front_caster" type="fixed">
-       <parent link="base_link"/>
-       <child link="front_caster"/>
-       <origin xyz="0 0.25 0.03" rpy="0 0 0"/>
-  </joint>
-   <link name="back_caster">
-  	<visual>
-  		<pose xyz="0 -0.25 0.03" rpy="0 0 0"/>
-  		<geometry>
-        	   <sphere radius="0.05"/>
-        	</geometry>
-        </visual>
-        <collision>
-        	<pose xyz="0 -0.25 0.03" rpy="0 0 0"/>
-  		<geometry>
-        	   <sphere radius="0.05"/>
-        	</geometry>
-        </collision>
-   </link>
-   <joint name="base_link_to_back_caster" type="fixed">
-      <parent link="base_link"/>
-      <child link="back_caster"/>
-      <origin xyz="0 -0.25 0.03" rpy="0 0 0"/>
-   </joint>
-   <link name="AGV_1/base_footprint"/>
-    <joint name="base_joint" type="fixed">
-       <parent link="AGV_1/base_footprint"/>
-       <child link="base_link"/>
-       <origin xyz="0 0 0" rpy="0 0 0"/>
-    </joint>
-   <link name="wheel_left">
-       <visual>
-          <origin xyz="0 0 0"  rpy="0 0 0" />
-          <geometry>
-      	     <cylinder radius="0.1" length="0.05"/>
-          </geometry>
-       </visual>
-       <collision>
-  	  <geometry>
-      	     <cylinder radius="0.1" length="0.05"/>
-        </geometry>
-       </collision>
-   </link>
-   <joint name="base_link_to_wheel_left" type="continuous">
-    <parent link="base_link"/>
-    <child link="wheel_left"/>
-    <axis xyz="0 0 1"/>
-    <origin xyz="-0.22 0.005 0.1" rpy="0 -1.57079633 0"/>
-  </joint>
-  <link name="wheel_right">
-     <visual>
-       <origin xyz="0 0 0" rpy="0 0 0" />
-        <geometry>
-      	 <cylinder radius="0.1" length="0.05"/>
-       </geometry>
-     </visual>
-     <collision>
-  	<geometry>
-         <cylinder radius="0.1" length="0.05"/>
-        </geometry>
-     </collision>
-   </link>
-   <joint name="base_link_to_wheel_right" type="continuous">
-    <parent link="base_link"/>
-    <child link="wheel_right"/>
-    <axis xyz="0 0 1"/>
-    <origin xyz="0.22 0.005 0.1" rpy="0 -1.57079633 0"/>
-  </joint>
-  <link name="laser_front">
-    <visual>
+  <link name="AGV_1/wheel_left">
+    <inertial>
+      <mass value="0"/>
+      <origin xyz="0 0 0" rpy="0 0 0"/>
+      <inertia ixx="0" ixy="0" ixz="0" iyy="0" iyz="0" izz="0"/>
+    </inertial>
+    <collision name="AGV_1/collision">
+      <origin xyz="0 0 0" rpy="0 0 0"/>
       <geometry>
-        <mesh
-          filename="package://itu_agv_description/meshes/lms200.dae" scale="0.001 0.001 0.001" />
-      </geometry>
-      <origin rpy="-1.57079633 0 3.14" xyz="0 0 0"/>
-    </visual>
-    <collision>
-      <geometry>
-        <mesh
-          filename="package://itu_agv_description/meshes/lms200.dae" scale="0.001 0.001 0.001" />
+        <cylinder radius=".1" length=".05"/>
       </geometry>
     </collision>
   </link>
-  <joint name="base_link_to_laser_front" type="fixed">
-    <parent link="base_link"/>
-    <child link="laser_front"/>
-    <origin xyz="0 0.4 0.305" rpy="0 0 0"/>
-  </joint>
-  <link name="laser_back">
-    <visual>
+  <link name="AGV_1/wheel_right">
+    <inertial>
+      <mass value="0"/>
+      <origin xyz="0 0 0" rpy="0 0 0"/>
+      <inertia ixx="0" ixy="0" ixz="0" iyy="0" iyz="0" izz="0"/>
+    </inertial>
+    <collision name="AGV_1/collision">
+      <origin xyz="0 0 0" rpy="0 0 0"/>
       <geometry>
-        <mesh
-        filename="package://itu_agv_description/meshes/lms200_2.dae" scale="0.001 0.001 0.001" />
+        <cylinder radius=".1" length=".05"/>
       </geometry>
-      <origin rpy="-1.57079633 0 0" xyz="-0.0775 -0.078 0.105"/>
-      <material name="blue"/>
-    </visual>
-    <collision>
-      <geometry>
-        <mesh
-        filename="package://itu_agv_description/meshes/lms200_2.dae" scale="0.001 0.001 0.001" />
-      </geometry>
-     </collision>
+    </collision>
   </link>
-  <joint name="base_link_to_laser_back" type="fixed">
-    <parent link="base_link"/>
-    <child link="laser_back"/>
-    <origin xyz="0 -0.4 0.305" rpy="0 0 3.14"/>
-  </joint>
-   <link name="platform">
-  	<visual>
-  	   <geometry>
-  	      <mesh
-  		filename="package://itu_agv_description/meshes/tabla.dae" />
-      	   </geometry>
-      	   <origin rpy="1.571 0 1.571" xyz="-0.925 0.13 -0.41"/>
-      	</visual>
-      	<collision>
-         <geometry>
-          <mesh
-          filename="package://itu_agv_description/meshes/tabla.dae" />
-         </geometry>
-      <origin rpy="1.571 0 1.571" xyz="-0.925 0.13 -0.41"/>
-      </collision>
-  </link>
-  <joint name="base_link_to_tabla" type="fixed">
-    <parent link="base_link"/>
-    <child link="platform"/>
-    <origin xyz="0 0 0.55" rpy="0 0 0"/>
-  </joint>
-  <link name="Velodyne">
-  	<visual>
-  	   <geometry>
-  	      <mesh
-  		filename="package://itu_agv_description/meshes/Velodyne.dae" />
-      	   </geometry>
-      	   <origin rpy="1.571 0 1.571" xyz="0 0 -0.05"/>
-      	</visual>
-      	<collision>
-      <geometry>
-        <mesh
-        filename="package://itu_agv_description/meshes/Velodyne.dae" />
-      </geometry>
-      <origin rpy="1.571 0 1.571" xyz="0 0 -0.05"/>
-      </collision>
-  </link>
-  <joint name="base_link_to_Velodyne" type="fixed">
-    <parent link="platform"/>
-    <child link="Velodyne"/>
-    <origin xyz="0 0 0.15" rpy="0 0 0"/>
-  </joint>
-  <link name="camera_link">
-  	<visual>
-  	   <geometry>
-  	      <mesh
-  		filename="package://itu_agv_description/meshes/Camera.dae" />
-      	   </geometry>
-      	   <origin rpy="-1.571 0 0" xyz="0 0 0"/>
-      	</visual>
-      	<collision>
-      <geometry>
-        <mesh
-        filename="package://itu_agv_description/meshes/Camera.dae" />
-      </geometry>
-     </collision>
-  </link>
-  <joint name="base_link_to_Camera" type="fixed">
-    <parent link="platform"/>
-    <child link="camera_link"/>
-    <origin xyz="0 0.125 0.03" rpy="0 0 0"/>
-  </joint>
-  <link name="IMU">
-  	<visual>
-  	   <geometry>
-  	      <mesh
-  		filename="package://itu_agv_description/meshes/IMU.dae" />
-      	   </geometry>
-      	   <origin rpy="0 0 0" xyz="0 0 0"/>
-      	</visual>
-      	<collision>
-      <geometry>
-        <mesh
-        filename="package://itu_agv_description/meshes/IMU.dae" />
-      </geometry>
-     </collision>
-  </link>
-  <joint name="base_link_to_IMU" type="fixed">
-    <parent link="base_link"/>
-    <child link="IMU"/>
-    <origin xyz="0 0 0.56" rpy="0 0 3.14"/>
-  </joint>
 </robot>
